File: PCB/HerbUnitPCB/ESP32_S3.kicad_sch (KiCad schematic)
At the start: 23 parts, among them J1 USB_C_Receptacle_USB2.0_16P, SW1 SW_Push, SW2 SW_Push, U1 USBLC6-2P6, U2 AP2112K-3.3, U3 ESP32-S3-WROOM-1

Commit message: Finished Baseline Electrical Schema
Parts:
- added C5: 10u, Capacitor_SMD:C_0402_1005Metric, symbol Device:C
- added J2: Barrel_Jack_Switch_Pin3Ring, Connector_BarrelJack:BarrelJack_Horizontal, symbol Connector:Barrel_Jack_Switch_Pin3Ring
- added U3: AMS1117-5.0, Package_TO_SOT_SMD:SOT-223-3_TabPin2, symbol Regulator_Linear:AMS1117-5.0
- renumbered C7 to C1, C8 to C2, C5 to C6, C6 to C7, C1 to C8, C2 to C9, R8 to R1, R6 to R2, R7 to R3, R1 to R4, R4 to R5, R2 to R6, R5 to R7, R3 to R8, U3 to U2, U2 to U4
Connections:
- net GND: now also C5.2, J2.3, U3.1 (GND)
- net +3.3V renamed +3.3V_USB
- net VBUS: no longer names the net of C3.1, D1.1 (K), J1.A4 (VBUS), J1.A9 (VBUS), J1.B4 (VBUS), J1.B9 (VBUS), R1.1
- new net: C5.1, J2.1, U3.3 (VI)
- new net +5V_JACK: U3.2 (VO)
- no-connect marks 23 -> 24
Other:
- note added: "5 LDO & Jack"
- note added: "USB-C & USB-C Power"
- note removed: "Power & USB-C"
