File: PCB/HerbUnitPCB/peripherals.kicad_sch (KiCad schematic)
At the start: 14 parts, among them J2 SD_Card_Device, J3 Conn_01x03_Pin, J4 Screw_Terminal_01x02, SW3 SW_Push, U4 DHT11

Commit message: Finished Baseline Electrical Schema
Parts:
- added J6: Conn_01x03_Pin, symbol Connector:Conn_01x03_Pin
- renumbered J2 to J4, J4 to J5, R9 to R10, R12 to R11, R10 to R12, R11 to R13, R13 to R9, U4 to U5
Connections:
- net GND: now also J6.1 (Pin_1)
- net SD_MOSI: no longer J4.7 (DAT0)
- net +3.3V renamed +3.3V_USB
- new net +5V_JACK: J6.2 (Pin_2)
- new net PumpMotor: J6.3 (Pin_3)
- new net SD_MISO: J4.7 (DAT0)
Other:
- note added: "Pump Header"
